Commit message: restored collisions

File: robots/go1.urdf.xacro (robot description, xacro)
@@ -43,4 +43,10 @@
             <!-- <material name="orange"/> -->
         </visual>
+        <collision>
+            <origin rpy="0 0 0" xyz="0 0 0"/>
+            <geometry>
+                <box size="${trunk_length} ${trunk_width} ${trunk_height}"/>
+            </geometry>
+        </collision>
         <inertial>
             <origin rpy="0 0 0" xyz="${trunk_com_x} ${trunk_com_y} ${trunk_com_z}"/>

File: urdfs/const.xacro (robot description, xacro)
@@ -29,20 +29,18 @@
     <xacro:property name="hip_offset" value="0.08"/>
     <!-- joint limits -->
-    <!-- xacro:property name="damping" value="0.01"/>
-    <xacro:property name="friction" value="0.2"/-->
-    <xacro:property name="damping" value="0.5"/>
-    <xacro:property name="friction" value="0.0"/>
-    <xacro:property name="haa_max" value="260"/>
-    <xacro:property name="haa_min" value="-260"/>
+    <xacro:property name="damping" value="0.01"/>
+    <xacro:property name="friction" value="0.2"/>
+    <xacro:property name="haa_max" value="60"/>
+    <xacro:property name="haa_min" value="-60"/>
     <xacro:property name="haa_velocity_max" value="30.1"/>
-    <xacro:property name="haa_torque_max" value="123.7"/>
-    <xacro:property name="hfe_max" value="270"/>
-    <xacro:property name="hfe_min" value="-238"/>
+    <xacro:property name="haa_torque_max" value="23.7"/>
+    <xacro:property name="hfe_max" value="170"/>
+    <xacro:property name="hfe_min" value="-38"/>
     <xacro:property name="hfe_velocity_max" value="30.1"/>
-    <xacro:property name="hfe_torque_max" value="123.7"/>
-    <xacro:property name="kfe_max" value="1000"/>
-    <xacro:property name="kfe_min" value="-2860"/>
+    <xacro:property name="hfe_torque_max" value="23.7"/>
+    <xacro:property name="kfe_max" value="-48"/>
+    <xacro:property name="kfe_min" value="-156"/>
     <xacro:property name="kfe_velocity_max" value="30.1"/>
-    <xacro:property name="kfe_torque_max" value="123.7"/>
+    <xacro:property name="kfe_torque_max" value="23.7"/>
     <!-- dynamics inertial value        total 12.84kg -->
     <!-- trunk -->

File: urdfs/leg.xacro (robot description, xacro)
@@ -10,5 +10,5 @@
             <child link="${name}_hip"/>
             <axis xyz="1 0 0"/>
-            <!--dynamics damping="${damping}" friction="${friction}"/-->
+            <dynamics damping="${damping}" friction="${friction}"/>
             <xacro:if value="${(mirror_dae == True)}">
                 <limit effort="${haa_torque_max}" velocity="${haa_velocity_max}" lower="${haa_min*PI/180.0}" upper="${haa_max*PI/180.0}"/>
@@ -37,4 +37,10 @@
                 <!-- <material name="orange"/> -->
             </visual>
+            <collision>
+                <origin rpy="${PI/2.0} 0 0" xyz="0 0 0"/>
+                <geometry>
+                    <cylinder length="${hip_length}" radius="${hip_radius}"/>
+                </geometry>
+            </collision>
             <inertial>
                 <origin rpy="0 0 0" xyz="${hip_com_x*front_hind} ${hip_com_y*mirror} ${hip_com_z}"/>
@@ -53,4 +59,10 @@
         <!-- this link is only for collision -->
         <link name="${name}_upperleg_shoulder">
+            <collision>
+                <origin rpy="${PI/2.0} 0 0" xyz="0 0 0"/>
+                <geometry>
+                    <cylinder length="${upperleg_shoulder_length}" radius="${upperleg_shoulder_radius}"/>
+                </geometry>
+            </collision>
         </link>
         <joint name="${name}_hfe_joint" type="revolute">
@@ -59,5 +71,5 @@
             <child link="${name}_upperleg"/>
             <axis xyz="0 1 0"/>
-            <!-- dynamics damping="${damping}" friction="${friction}"/ -->
+            <dynamics damping="${damping}" friction="${friction}"/>
             <limit effort="${hfe_torque_max}" velocity="${hfe_velocity_max}" lower="${hfe_min*PI/180.0}" upper="${hfe_max*PI/180.0}"/>
         </joint>
@@ -75,4 +87,10 @@
                 <!-- <material name="orange"/> -->
             </visual>
+            <collision>
+                <origin rpy="0 ${PI/2.0} 0" xyz="0 0 ${-upperleg_length/2.0}"/>
+                <geometry>
+                    <box size="${upperleg_length} ${upperleg_width} ${upperleg_height}"/>
+                </geometry>
+            </collision>
             <inertial>
                 <origin rpy="0 0 0" xyz="${upperleg_com_x} ${upperleg_com_y*mirror} ${upperleg_com_z}"/>
@@ -89,5 +107,5 @@
             <child link="${name}_lowerleg"/>
             <axis xyz="0 1 0"/>
-            <!-- dynamics damping="${damping}" friction="${friction}"/-->
+            <dynamics damping="${damping}" friction="${friction}"/>
             <limit effort="${kfe_torque_max}" velocity="${kfe_velocity_max}" lower="${kfe_min*PI/180.0}" upper="${kfe_max*PI/180.0}"/>
         </joint>
@@ -100,4 +118,10 @@
                 <!-- <material name="orange"/> -->
             </visual>
+            <collision>
+                <origin rpy="0 ${PI/2.0} 0" xyz="0 0 ${-lowerleg_length/2.0}"/>
+                <geometry>
+                    <box size="${lowerleg_length} ${lowerleg_width} ${lowerleg_height}"/>
+                </geometry>
+            </collision>
             <inertial>
                 <origin rpy="0 0 0" xyz="${lowerleg_com_x} ${lowerleg_com_y} ${lowerleg_com_z}"/>
@@ -118,8 +142,14 @@
                 <origin rpy="0 0 0" xyz="0 0 0"/>
                 <geometry>
-                    <sphere radius="${foot_radius}"/>
+                    <sphere radius="${foot_radius-0.01}"/>
                 </geometry>
                 <!-- <material name="orange"/> -->
             </visual>
+            <collision>
+                <origin rpy="0 0 0" xyz="0 0 0"/>
+                <geometry>
+                    <sphere radius="${foot_radius}"/>
+                </geometry>
+            </collision>
             <inertial>
                 <mass value="${foot_mass}"/>
