Commit message: finding a solution for angles singularity when crossing pi

File: robots/go1.srdf.xacro (robot description, xacro)
@@ -44,28 +44,28 @@
 	    <joint name="lf_haa_joint" value="0.20" />
 	    <joint name="lf_hfe_joint" value="0.78" />
-	    <joint name="lf_kfe_joint" value="-1.57" />
+	    <joint name="lf_kfe_joint" value="-1.7" />
 	    <joint name="lh_haa_joint" value="0.20" />
 	    <joint name="lh_hfe_joint" value="0.78" />
-	    <joint name="lh_kfe_joint" value="-1.57" />
+	    <joint name="lh_kfe_joint" value="-1.7" />
 	    <joint name="rf_haa_joint" value="-0.20" />
 	    <joint name="rf_hfe_joint" value="0.78" />
-	    <joint name="rf_kfe_joint" value="-1.57" />
+	    <joint name="rf_kfe_joint" value="-1.7" />
 	    <joint name="rh_haa_joint" value="-0.2" />
 	    <joint name="rh_hfe_joint" value="0.78" />
-	    <joint name="rh_kfe_joint" value="-1.57" />
+	    <joint name="rh_kfe_joint" value="-1.7" />
 	</group_state>
-	<group_state group="chains" name="standdown">
+	<group_state group="chains" name="home">
         <joint name="lf_haa_joint" value="0.60"/>
         <joint name="lf_hfe_joint" value="1.70"/>
-        <joint name="lf_kfe_joint" value="-2.77"/>
+        <joint name="lf_kfe_joint" value="3.7"/>
         <joint name="lh_haa_joint" value="0.60"/>
         <joint name="lh_hfe_joint" value="1.52"/>
-        <joint name="lh_kfe_joint" value="-2.77"/>
+        <joint name="lh_kfe_joint" value="3.7"/>
         <joint name="rf_haa_joint" value="-0.60"/>
         <joint name="rf_hfe_joint" value="1.70"/>
-        <joint name="rf_kfe_joint" value="-2.77"/>
+        <joint name="rf_kfe_joint" value="3.7"/>
         <joint name="rh_haa_joint" value="-0.60"/>
         <joint name="rh_hfe_joint" value="1.52"/>
-        <joint name="rh_kfe_joint" value="-2.77"/>
+        <joint name="rh_kfe_joint" value="3.7"/>
     </group_state>
 </robot>

File: robots/go1.urdf.xacro (robot description, xacro)
@@ -43,10 +43,4 @@
             <!-- <material name="orange"/> -->
         </visual>
-        <collision>
-            <origin rpy="0 0 0" xyz="0 0 0"/>
-            <geometry>
-                <box size="${trunk_length} ${trunk_width} ${trunk_height}"/>
-            </geometry>
-        </collision>
         <inertial>
             <origin rpy="0 0 0" xyz="${trunk_com_x} ${trunk_com_y} ${trunk_com_z}"/>

File: urdfs/const.xacro (robot description, xacro)
@@ -29,18 +29,20 @@
     <xacro:property name="hip_offset" value="0.08"/>
     <!-- joint limits -->
-    <xacro:property name="damping" value="0.01"/>
-    <xacro:property name="friction" value="0.2"/>
-    <xacro:property name="haa_max" value="60"/>
-    <xacro:property name="haa_min" value="-60"/>
+    <!-- xacro:property name="damping" value="0.01"/>
+    <xacro:property name="friction" value="0.2"/-->
+    <xacro:property name="damping" value="0.5"/>
+    <xacro:property name="friction" value="0.0"/>
+    <xacro:property name="haa_max" value="260"/>
+    <xacro:property name="haa_min" value="-260"/>
     <xacro:property name="haa_velocity_max" value="30.1"/>
-    <xacro:property name="haa_torque_max" value="23.7"/>
-    <xacro:property name="hfe_max" value="170"/>
-    <xacro:property name="hfe_min" value="-38"/>
+    <xacro:property name="haa_torque_max" value="123.7"/>
+    <xacro:property name="hfe_max" value="270"/>
+    <xacro:property name="hfe_min" value="-238"/>
     <xacro:property name="hfe_velocity_max" value="30.1"/>
-    <xacro:property name="hfe_torque_max" value="23.7"/>
-    <xacro:property name="kfe_max" value="-48"/>
-    <xacro:property name="kfe_min" value="-156"/>
+    <xacro:property name="hfe_torque_max" value="123.7"/>
+    <xacro:property name="kfe_max" value="1000"/>
+    <xacro:property name="kfe_min" value="-2860"/>
     <xacro:property name="kfe_velocity_max" value="30.1"/>
-    <xacro:property name="kfe_torque_max" value="23.7"/>
+    <xacro:property name="kfe_torque_max" value="123.7"/>
     <!-- dynamics inertial value        total 12.84kg -->
     <!-- trunk -->

File: urdfs/leg.gazebo.xacro (robot description, xacro)
@@ -21,72 +21,33 @@
 		    </visual>
 	    </gazebo-->
-        <!-- GAZEBO-NATIVE PLUGINS -->
-        <gazebo reference="${name}_haa_joint">
-            <provideFeedback>true</provideFeedback>
-        </gazebo>
-        <gazebo reference="${name}_kfe_joint">
-            <provideFeedback>true</provideFeedback>
-        </gazebo>
-        <gazebo reference="${name}_hfe_joint">
-            <provideFeedback>true</provideFeedback>
-        </gazebo>
-        <xacro:if value="${load_force_sensors}">
-            <gazebo>
-                <plugin name="${name}_haa_sensor" filename="libgazebo_ros_ft_sensor.so">
-                    <robotNamespace>/internal_wrench/</robotNamespace>
-                    <updateRate>100.0</updateRate>
-                    <topicName>${name}_haa_joint</topicName>
-                    <jointName>${name}_haa_joint</jointName>
-                </plugin>
-            </gazebo>
-            <gazebo>
-                <plugin name="${name}_kfe_sensor" filename="libgazebo_ros_ft_sensor.so">
-                    <robotNamespace>/internal_wrench/</robotNamespace>
-                    <updateRate>100.0</updateRate>
-                    <topicName>${name}_kfe_joint</topicName>
-                    <jointName>${name}_kfe_joint</jointName>
-                </plugin>
-            </gazebo>
-            <gazebo>
-                <plugin name="${name}_hfe_sensor" filename="libgazebo_ros_ft_sensor.so">
-                    <robotNamespace>/internal_wrench/</robotNamespace>
-                    <updateRate>100.0</updateRate>
-                    <topicName>${name}_hfe_joint</topicName>
-                    <jointName>${name}_hfe_joint</jointName>
-                </plugin>
-            </gazebo>
-        </xacro:if>
-        <gazebo reference="${name}_hip">
-		    <mu1>0.2</mu1>
-    		<mu2>0.2</mu2>
-    		<material>Gazebo/DarkGrey</material>
-	    </gazebo>
-	    <gazebo reference="${name}_upperleg">
-	    	<mu1>0.2</mu1>
-	    	<mu2>0.2</mu2>
-	    	<self_collide>1</self_collide>
-	    	<material>Gazebo/DarkGrey</material>
-	    	<kp  value="1000000.0"/>
-	    	<kd  value="1.0"/>
-	    </gazebo>
-	    <gazebo reference="${name}_lowerleg">
-	    	<mu1>0.2</mu1>
-	    	<mu2>0.2</mu2>
-	    	<self_collide>1</self_collide>
-	    </gazebo>
+		<gazebo reference="${name}_upperleg">
+			<kp>1000000.0</kp>
+			<kd>100.0</kd>
+			<mu1>1.5</mu1>
+			<mu2>1.5</mu2>
+			<fdir1>1 0 0</fdir1>
+			<maxVel>1.0</maxVel>
+			<minDepth>0.00</minDepth>
+		</gazebo>
+		<gazebo reference="${name}_lowerleg">
+			<kp>1000000.0</kp>
+			<kd>100.0</kd>
+			<mu1>1.0</mu1>
+			<mu2>1.0</mu2>
+			<maxVel>1.0</maxVel>
+			<maxContacts>1</maxContacts>
+		</gazebo>
         <gazebo reference="${name}_foot">
-            <mu1>0.6</mu1>
-	    	<mu2>0.6</mu2>
-	    	<self_collide>1</self_collide>
-	    	<material>Gazebo/DarkGrey</material>
-	    	<kp  value="1000000.0"/>
-	    	<kd  value="1.0"/>
+            <kp>1000000.0</kp>
+            <kd>100.0</kd>
+            <mu1>1.0</mu1>
+            <mu2>1.0</mu2>
             <maxVel>1.0</maxVel>
-            <maxContacts>1</maxContacts>
+			<maxContacts>1</maxContacts>
             <sensor name="${name}_foot_contact_sensor" type="contact">
                 <always_on>true</always_on>
                 <update_rate>1000.0</update_rate>
                 <contact>
-                    <collision>${name}_lower_leg_fixed_joint_lump__${name}_foot_collision_1</collision>
+                    <collision>${name}_lowerleg_fixed_joint_lump__${name}_foot_collision_1</collision>
                 </contact>
                 <!-- the sensor readings in terms of force torques are expressed in the lowerleg frame

File: urdfs/leg.xacro (robot description, xacro)
@@ -10,5 +10,5 @@
             <child link="${name}_hip"/>
             <axis xyz="1 0 0"/>
-            <dynamics damping="${damping}" friction="${friction}"/>
+            <!--dynamics damping="${damping}" friction="${friction}"/-->
             <xacro:if value="${(mirror_dae == True)}">
                 <limit effort="${haa_torque_max}" velocity="${haa_velocity_max}" lower="${haa_min*PI/180.0}" upper="${haa_max*PI/180.0}"/>
@@ -37,10 +37,4 @@
                 <!-- <material name="orange"/> -->
             </visual>
-            <collision>
-                <origin rpy="${PI/2.0} 0 0" xyz="0 0 0"/>
-                <geometry>
-                    <cylinder length="${hip_length}" radius="${hip_radius}"/>
-                </geometry>
-            </collision>
             <inertial>
                 <origin rpy="0 0 0" xyz="${hip_com_x*front_hind} ${hip_com_y*mirror} ${hip_com_z}"/>
@@ -59,10 +53,4 @@
         <!-- this link is only for collision -->
         <link name="${name}_upperleg_shoulder">
-            <collision>
-                <origin rpy="${PI/2.0} 0 0" xyz="0 0 0"/>
-                <geometry>
-                    <cylinder length="${upperleg_shoulder_length}" radius="${upperleg_shoulder_radius}"/>
-                </geometry>
-            </collision>
         </link>
         <joint name="${name}_hfe_joint" type="revolute">
@@ -71,5 +59,5 @@
             <child link="${name}_upperleg"/>
             <axis xyz="0 1 0"/>
-            <dynamics damping="${damping}" friction="${friction}"/>
+            <!-- dynamics damping="${damping}" friction="${friction}"/ -->
             <limit effort="${hfe_torque_max}" velocity="${hfe_velocity_max}" lower="${hfe_min*PI/180.0}" upper="${hfe_max*PI/180.0}"/>
         </joint>
@@ -87,10 +75,4 @@
                 <!-- <material name="orange"/> -->
             </visual>
-            <collision>
-                <origin rpy="0 ${PI/2.0} 0" xyz="0 0 ${-upperleg_length/2.0}"/>
-                <geometry>
-                    <box size="${upperleg_length} ${upperleg_width} ${upperleg_height}"/>
-                </geometry>
-            </collision>
             <inertial>
                 <origin rpy="0 0 0" xyz="${upperleg_com_x} ${upperleg_com_y*mirror} ${upperleg_com_z}"/>
@@ -107,5 +89,5 @@
             <child link="${name}_lowerleg"/>
             <axis xyz="0 1 0"/>
-            <dynamics damping="${damping}" friction="${friction}"/>
+            <!-- dynamics damping="${damping}" friction="${friction}"/-->
             <limit effort="${kfe_torque_max}" velocity="${kfe_velocity_max}" lower="${kfe_min*PI/180.0}" upper="${kfe_max*PI/180.0}"/>
         </joint>
@@ -118,10 +100,4 @@
                 <!-- <material name="orange"/> -->
             </visual>
-            <collision>
-                <origin rpy="0 ${PI/2.0} 0" xyz="0 0 ${-lowerleg_length/2.0}"/>
-                <geometry>
-                    <box size="${lowerleg_length} ${lowerleg_width} ${lowerleg_height}"/>
-                </geometry>
-            </collision>
             <inertial>
                 <origin rpy="0 0 0" xyz="${lowerleg_com_x} ${lowerleg_com_y} ${lowerleg_com_z}"/>
@@ -142,14 +118,8 @@
                 <origin rpy="0 0 0" xyz="0 0 0"/>
                 <geometry>
-                    <sphere radius="${foot_radius-0.01}"/>
+                    <sphere radius="${foot_radius}"/>
                 </geometry>
                 <!-- <material name="orange"/> -->
             </visual>
-            <collision>
-                <origin rpy="0 0 0" xyz="0 0 0"/>
-                <geometry>
-                    <sphere radius="${foot_radius}"/>
-                </geometry>
-            </collision>
             <inertial>
                 <mass value="${foot_mass}"/>

Commit message: IMPORTANT! there is a bug in set_model_configuration
if you set angle <-2.2 it returns the 2*pi - angle!

File: robots/go1.srdf.xacro (robot description, xacro)
@@ -56,16 +56,16 @@
 	</group_state>
 	<group_state group="chains" name="home">
-        <joint name="lf_haa_joint" value="0.60"/>
+        <joint name="lf_haa_joint" value="0.80"/>
         <joint name="lf_hfe_joint" value="1.70"/>
-        <joint name="lf_kfe_joint" value="3.7"/>
-        <joint name="lh_haa_joint" value="0.60"/>
+        <joint name="lf_kfe_joint" value="-2."/>
+        <joint name="lh_haa_joint" value="0.80"/>
         <joint name="lh_hfe_joint" value="1.52"/>
-        <joint name="lh_kfe_joint" value="3.7"/>
-        <joint name="rf_haa_joint" value="-0.60"/>
+        <joint name="lh_kfe_joint" value="-2."/>
+        <joint name="rf_haa_joint" value="-0.80"/>
         <joint name="rf_hfe_joint" value="1.70"/>
-        <joint name="rf_kfe_joint" value="3.7"/>
-        <joint name="rh_haa_joint" value="-0.60"/>
+        <joint name="rf_kfe_joint" value="-2."/>
+        <joint name="rh_haa_joint" value="-0.80"/>
         <joint name="rh_hfe_joint" value="1.52"/>
-        <joint name="rh_kfe_joint" value="3.7"/>
+        <joint name="rh_kfe_joint" value="-2."/>
     </group_state>
 </robot>

File: robots/go1.urdf.xacro (robot description, xacro)
@@ -44,5 +44,5 @@
         </visual>
         <collision>
-            <origin rpy="0 0 0" xyz="0 0 0"/>
+            <origin rpy="0 0 0" xyz="0 0 -0.05"/>
             <geometry>
                 <box size="${trunk_length} ${trunk_width} ${trunk_height}"/>

Commit message: lh_hfe_joint value corrected

File: robots/go1.srdf.xacro (robot description, xacro)
@@ -60,5 +60,5 @@
         <joint name="lf_kfe_joint" value="-2."/>
         <joint name="lh_haa_joint" value="0.80"/>
-        <joint name="lh_hfe_joint" value="1.52"/>
+        <joint name="lh_hfe_joint" value="1.70"/>
         <joint name="lh_kfe_joint" value="-2."/>
         <joint name="rf_haa_joint" value="-0.80"/>
@@ -66,5 +66,5 @@
         <joint name="rf_kfe_joint" value="-2."/>
         <joint name="rh_haa_joint" value="-0.80"/>
-        <joint name="rh_hfe_joint" value="1.52"/>
+        <joint name="rh_hfe_joint" value="1.70"/>
         <joint name="rh_kfe_joint" value="-2."/>
     </group_state>
