Commit message: restored torque limits

File: urdfs/const.xacro (robot description, xacro)
@@ -44,13 +44,13 @@
     <xacro:property name="haa_min" value="-360"/>
     <xacro:property name="haa_velocity_max" value="3000"/>
-    <xacro:property name="haa_torque_max" value="2370"/>
+    <xacro:property name="haa_torque_max" value="23.70"/>
     <xacro:property name="hfe_max" value="360"/>
     <xacro:property name="hfe_min" value="-360"/>
     <xacro:property name="hfe_velocity_max" value="3000"/>
-    <xacro:property name="hfe_torque_max" value="2370"/>
+    <xacro:property name="hfe_torque_max" value="23.70"/>
     <xacro:property name="kfe_max" value="360"/>
     <xacro:property name="kfe_min" value="-360"/>
     <xacro:property name="kfe_velocity_max" value="3000"/>
-    <xacro:property name="kfe_torque_max" value="2370"/>
+    <xacro:property name="kfe_torque_max" value="23.70"/>
     <!-- dynamics inertial value        total 12.84kg -->
     <!-- trunk -->

Commit message: restore joint limits

File: urdfs/const.xacro (robot description, xacro)
@@ -41,16 +41,16 @@
     <xacro:property name="damping" value="0.00"/>
     <xacro:property name="friction" value="0.0"/>
-    <xacro:property name="haa_max" value="360"/>
-    <xacro:property name="haa_min" value="-360"/>
-    <xacro:property name="haa_velocity_max" value="3000"/>
-    <xacro:property name="haa_torque_max" value="23.70"/>
-    <xacro:property name="hfe_max" value="360"/>
-    <xacro:property name="hfe_min" value="-360"/>
-    <xacro:property name="hfe_velocity_max" value="3000"/>
-    <xacro:property name="hfe_torque_max" value="23.70"/>
-    <xacro:property name="kfe_max" value="360"/>
-    <xacro:property name="kfe_min" value="-360"/>
-    <xacro:property name="kfe_velocity_max" value="3000"/>
-    <xacro:property name="kfe_torque_max" value="23.70"/>
+    <xacro:property name="haa_max" value="0.863"/>
+    <xacro:property name="haa_min" value="-0.863"/>
+    <xacro:property name="haa_velocity_max" value="30.1"/>
+    <xacro:property name="haa_torque_max" value="23.7"/>
+    <xacro:property name="hfe_max" value="4.501"/>
+    <xacro:property name="hfe_min" value="-0.686"/>
+    <xacro:property name="hfe_velocity_max" value="30.1"/>
+    <xacro:property name="hfe_torque_max" value="23.7"/>
+    <xacro:property name="kfe_max" value="-0.888"/>
+    <xacro:property name="kfe_min" value="-2.818"/>
+    <xacro:property name="kfe_velocity_max" value="20.06"/>
+    <xacro:property name="kfe_torque_max" value="35.55"/>
     <!-- dynamics inertial value        total 12.84kg -->
     <!-- trunk -->

File: urdfs/leg.xacro (robot description, xacro)
@@ -12,8 +12,8 @@
             <dynamics damping="${damping}" friction="${friction}"/>
             <xacro:if value="${(mirror_dae == True)}">
-                <limit effort="${haa_torque_max}" velocity="${haa_velocity_max}" lower="${haa_min*PI/180.0}" upper="${haa_max*PI/180.0}"/>
+                <limit effort="${haa_torque_max}" velocity="${haa_velocity_max}" lower="${haa_min}" upper="${haa_max}"/>
             </xacro:if>
             <xacro:if value="${(mirror_dae == False)}">
-                <limit effort="${haa_torque_max}" velocity="${haa_velocity_max}" lower="${-haa_max*PI/180.0}" upper="${-haa_min*PI/180.0}"/>
+                <limit effort="${haa_torque_max}" velocity="${haa_velocity_max}" lower="${-haa_max}" upper="${-haa_min}"/>
             </xacro:if>
         </joint>
@@ -112,5 +112,5 @@
             <axis xyz="0 1 0"/>
             <dynamics damping="${damping}" friction="${friction}"/>
-            <limit effort="${hfe_torque_max}" velocity="${hfe_velocity_max}" lower="${hfe_min*PI/180.0}" upper="${hfe_max*PI/180.0}"/>
+            <limit effort="${hfe_torque_max}" velocity="${hfe_velocity_max}" lower="${hfe_min}" upper="${hfe_max}"/>
         </joint>
         <!-- hfe motor -->
@@ -188,5 +188,5 @@
             <axis xyz="0 1 0"/>
             <dynamics damping="${damping}" friction="${friction}"/>
-            <limit effort="${kfe_torque_max}" velocity="${kfe_velocity_max}" lower="${kfe_min*PI/180.0}" upper="${kfe_max*PI/180.0}"/>
+            <limit effort="${kfe_torque_max}" velocity="${kfe_velocity_max}" lower="${kfe_min}" upper="${kfe_max}"/>
         </joint>
         <link name="${name}_lowerleg">

Commit message: rnlarged collision box (in this way it contains all the body+face+haa hind)

File: urdfs/const.xacro (robot description, xacro)
@@ -5,7 +5,11 @@
     <xacro:property name="stick_mass" value="0.00001"/>
     <!-- simplified collision value -->
-    <xacro:property name="trunk_width" value="0.0935"/>
+    <!--xacro:property name="trunk_width" value="0.0935"/>
     <xacro:property name="trunk_length" value="0.3762"/>
-    <xacro:property name="trunk_height" value="0.114"/>
+    <xacro:property name="trunk_height" value="0.114"/-->
+    <!--trunk artificially enlarged for colliions detection -->
+    <xacro:property name="trunk_width" value="0.22"/>
+    <xacro:property name="trunk_length" value="0.52"/>
+    <xacro:property name="trunk_height" value="0.14"/>
     <xacro:property name="hip_radius" value="0.046"/>
     <xacro:property name="hip_length" value="0.04"/>

Commit message: trunk resized for testing collisions

File: urdfs/const.xacro (robot description, xacro)
@@ -9,6 +9,6 @@
     <xacro:property name="trunk_height" value="0.114"/-->
     <!--trunk artificially enlarged for colliions detection -->
-    <xacro:property name="trunk_width" value="0.22"/>
-    <xacro:property name="trunk_length" value="0.52"/>
+    <xacro:property name="trunk_width" value="0.10"/>
+    <xacro:property name="trunk_length" value="0.45"/>
     <xacro:property name="trunk_height" value="0.14"/>
     <xacro:property name="hip_radius" value="0.046"/>
